File: PCB/FishShocker9000/_autosave-FishShocker9000.kicad_sch (KiCad schematic)
At the start: 160 parts, among them J1 Barrel_Jack, J10 P70-1000045R, J11 P70-1000045R, J12 P70-1000045R, J13 P70-1000045R, J14 P70-1000045R, J15 P70-1000045R, J16 P70-1000045R, J17 P70-1000045R, J18 P70-1000045R, J19 P70-1000045R, J20 P70-1000045R, J21 P70-1000045R, J22 P70-1000045R, J23 P70-1000045R, J24 P70-1000045R, J25 P70-1000045R, J26 P70-1000045R, J27 P70-1000045R, J28 P70-1000045R, J29 P70-1000045R, J3 P70-1000045R, J30 P70-1000045R, J31 P70-1000045R, J32 P70-1000045R, J33 P70-1000045R, J34 P70-1000045R, J35 P70-1000045R, J36 P70-1000045R, J37 P70-1000045R, J38 P70-1000045R, J39 P70-1000045R, J4 P70-1000045R, J40 P70-1000045R, J41 P70-1000045R, J42 P70-1000045R, J43 P70-1000045R, J44 P70-1000045R, J45 P70-1000045R, J46 P70-1000045R, J47 P70-1000045R, J48 P70-1000045R, J49 P70-1000045R, J5 P70-1000045R, J50 P70-1000045R, J51 P70-1000045R, J52 P70-1000045R, J53 P70-1000045R, J54 P70-1000045R, J55 P70-1000045R, J56 P70-1000045R, J57 P70-1000045R, J58 P70-1000045R, J59 P70-1000045R, J6 P70-1000045R, J60 P70-1000045R, J61 P70-1000045R, J62 P70-1000045R, J63 P70-1000045R, J64 P70-1000045R, J65 P70-1000045R, J66 P70-1000045R, J67 P70-1000045R, J68 P70-1000045R, J69 P70-1000045R, J7 P70-1000045R, J70 P70-1000045R, J71 P70-1000045R, J72 P70-1000045R, J73 P70-1000045R, J74 P70-1000045R, J75 Screw_Terminal_01x02, J8 P70-1000045R, J9 P70-1000045R, Q2 FQP27P06, U10 SN754410NE, U11 SN754410NE, U12 SN754410NE, U13 SN754410NE, U14 SN754410NE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

Commit message: New draft of final PCB layout
Parts:
- added Q1: IRLZ44N, Package_TO_SOT_THT:TO-220-3_Vertical, symbol Transistor_FET:IRLZ44N
- R7: value 220 -> 330
Connections:
- net BUCK_PG: now also Q1.1 (G); no longer D1.2 (A)
- net BUCK_VOUT: now also R7.2
- net GND: now also Q1.3 (S); no longer R7.1
- net at D1.1 (K): now also Q1.2 (D); no longer R7.2
- new net: D1.2 (A), R7.1
Other:
- moved on the sheet: D1, R1, R7
