File: PCB/FishShocker9000/FishShocker9000.kicad_sch (KiCad schematic)
At the start: 160 parts, among them J1 Barrel_Jack, J10 P70-1000045R, J11 P70-1000045R, J12 P70-1000045R, J13 P70-1000045R, J14 P70-1000045R, J15 P70-1000045R, J16 P70-1000045R, J17 P70-1000045R, J18 P70-1000045R, J19 P70-1000045R, J20 P70-1000045R, J21 P70-1000045R, J22 P70-1000045R, J23 P70-1000045R, J24 P70-1000045R, J25 P70-1000045R, J26 P70-1000045R, J27 P70-1000045R, J28 P70-1000045R, J29 P70-1000045R, J3 P70-1000045R, J30 P70-1000045R, J31 P70-1000045R, J32 P70-1000045R, J33 P70-1000045R, J34 P70-1000045R, J35 P70-1000045R, J36 P70-1000045R, J37 P70-1000045R, J38 P70-1000045R, J39 P70-1000045R, J4 P70-1000045R, J40 P70-1000045R, J41 P70-1000045R, J42 P70-1000045R, J43 P70-1000045R, J44 P70-1000045R, J45 P70-1000045R, J46 P70-1000045R, J47 P70-1000045R, J48 P70-1000045R, J49 P70-1000045R, J5 P70-1000045R, J50 P70-1000045R, J51 P70-1000045R, J52 P70-1000045R, J53 P70-1000045R, J54 P70-1000045R, J55 P70-1000045R, J56 P70-1000045R, J57 P70-1000045R, J58 P70-1000045R, J59 P70-1000045R, J6 P70-1000045R, J60 P70-1000045R, J61 P70-1000045R, J62 P70-1000045R, J63 P70-1000045R, J64 P70-1000045R, J65 P70-1000045R, J66 P70-1000045R, J67 P70-1000045R, J68 P70-1000045R, J69 P70-1000045R, J7 P70-1000045R, J70 P70-1000045R, J71 P70-1000045R, J72 P70-1000045R, J73 P70-1000045R, J74 P70-1000045R, J75 Screw_Terminal_01x02, J8 P70-1000045R, J9 P70-1000045R, Q2 FQP27P06, U10 SN754410NE, U11 SN754410NE, U12 SN754410NE, U13 SN754410NE, U14 SN754410NE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

Commit message: Changed Layout to eb more clean
Parts:
- added Q1: IRLZ44N, Package_TO_SOT_THT:TO-220-3_Vertical, symbol Transistor_FET:IRLZ44N
- R7: value 220 -> 330
Connections:
- net BUCK_PG: now also Q1.1 (G); no longer D1.2 (A)
- net BUCK_VOUT: now also R7.2
- net CELL1: now also U2.10 (3A); no longer U2.2 (1A)
- net CELL10: now also U13.2 (1A); no longer U13.10 (3A)
- net CELL11: now also U14.10 (3A); no longer U14.2 (1A)
- net CELL12: now also U14.2 (1A); no longer U14.10 (3A)
- net CELL2: now also U2.2 (1A); no longer U2.10 (3A)
- net CELL3: now also U10.10 (3A); no longer U10.2 (1A)
- net CELL4: now also U10.2 (1A); no longer U10.10 (3A)
- net CELL5: now also U11.10 (3A); no longer U11.2 (1A)
- net CELL6: now also U11.2 (1A); no longer U11.10 (3A)
- net CELL7: now also U12.10 (3A); no longer U12.2 (1A)
- net CELL8: now also U12.2 (1A); no longer U12.10 (3A)
- net CELL9: now also U13.10 (3A); no longer U13.2 (1A)
- net GND: now also Q1.3 (S); no longer R7.1
- net Plate 1.1: now also U2.14 (4Y); no longer U2.3 (1Y)
- net Plate 1.2: now also U2.11 (3Y); no longer U2.6 (2Y)
- net Plate 10.1: now also U13.6 (2Y); no longer U13.11 (3Y)
- net Plate 10.2: now also U13.3 (1Y); no longer U13.14 (4Y)
- net Plate 11.1: now also U14.14 (4Y); no longer U14.3 (1Y)
- net Plate 11.2: now also U14.11 (3Y); no longer U14.6 (2Y)
- net Plate 12.1: now also U14.6 (2Y); no longer U14.11 (3Y)
- net Plate 12.2: now also U14.3 (1Y); no longer U14.14 (4Y)
- net Plate 2.1: now also U2.6 (2Y); no longer U2.11 (3Y)
- net Plate 2.2: now also U2.3 (1Y); no longer U2.14 (4Y)
- net Plate 3.1: now also U10.14 (4Y); no longer U10.3 (1Y)
- net Plate 3.2: now also U10.11 (3Y); no longer U10.6 (2Y)
- net Plate 4.1: now also U10.6 (2Y); no longer U10.11 (3Y)
- net Plate 4.2: now also U10.3 (1Y); no longer U10.14 (4Y)
- net Plate 5.1: now also U11.14 (4Y); no longer U11.3 (1Y)
- net Plate 5.2: now also U11.11 (3Y); no longer U11.6 (2Y)
- net Plate 6.1: now also U11.6 (2Y); no longer U11.11 (3Y)
- net Plate 6.2: now also U11.3 (1Y); no longer U11.14 (4Y)
- net Plate 7.1: now also U12.14 (4Y); no longer U12.3 (1Y)
- net Plate 7.2: now also U12.11 (3Y); no longer U12.6 (2Y)
- net Plate 8.1: now also U12.6 (2Y); no longer U12.11 (3Y)
- net Plate 8.2: now also U12.3 (1Y); no longer U12.14 (4Y)
- net Plate 9.1: now also U13.14 (4Y); no longer U13.3 (1Y)
- net Plate 9.2: now also U13.11 (3Y); no longer U13.6 (2Y)
- net at D1.1 (K): now also Q1.2 (D); no longer R7.2
- new net: D1.2 (A), R7.1
Other:
- moved on the sheet: D1, R1, R7

Commit message: added various items to the schematic
Parts:
- removed J75: Screw_Terminal_01x02, TerminalBlock:TerminalBlock_Altech_AK300-2_P5.00mm, symbol Connector:Screw_Terminal_01x02
- removed R20, R21, R24, R26, R28, R30: 3.3k, Resistor_SMD:R_0805_2012Metric, symbol Device:R_Small
- removed R22, R23, R25, R27, R29, R31: 15k, Resistor_SMD:R_0805_2012Metric, symbol Device:R_Small
- removed R32, R33, R34, R35, R36, R37, R38, R39, R40, R41, R42, R43: 220, Resistor_SMD:R_0805_2012Metric, symbol Device:R_Small
- removed U10, U11, U12, U13, U14, U2: SN754410NE, Package_DIP:DIP-16_W7.62mm, symbol Driver_Motor:SN754410NE
- removed U15: TCAN334, Library:D0008A_L, symbol Interface_CAN_LIN:TCAN334
- removed U4, U5, U6, U7, U8, U9: OPA2197xD, Package_SO:SOIC-8_3.9x4.9mm_P1.27mm, symbol Amplifier_Operational:OPA2197xD
- added R48: 4.7k, Resistor_THT:R_Bare_Metal_Element_L12.4mm_W4.8mm_P11.40mm, symbol Device:R_Small_US
- added R49: 15k, Resistor_THT:R_Bare_Metal_Element_L12.4mm_W4.8mm_P11.40mm, symbol Device:R_Small_US
- added U19: DAC5311xDCK, Package_TO_SOT_SMD:SOT-363_SC-70-6, symbol Analog_DAC:DAC5311xDCK
- added U20: OPA197xD, Package_SO:SOIC-8_3.9x4.9mm_P1.27mm, symbol Amplifier_Operational:OPA197xD
- added U23, U24, U25, U26, U29, U30: SN754410NE, Package_DIP:DIP-16_W7.62mm, symbol Driver_Motor:SN754410NE
- D10, D11, D12, D13, D2, D3, D4, D5, D6, D7, D8, D9: value GREEN -> LED
- R10, R12, R14, R16, R17, R8: value 3.3k -> 220
- R11, R13, R15, R18, R19, R9: value 15k -> 220
Connections:
- net CELL1 is gone; now on net A1: R9.1
- net CELL2 is gone; now on net A5: R11.1
- net CELL3 is gone; now on net A9: R13.1
- net CELL4 is gone; now on net A6: R15.1
- net CELL5 is gone; now on net A7: R18.1
- net CELL7 is gone; now on net A11: R19.1
- net A0: now also R8.1, U23.1 (1,2EN)
- net A1: now also U23.9 (3,4EN)
- net A10: now also R16.1, U30.1 (1,2EN)
- net A11: now also U30.9 (3,4EN)
- net A2: now also R14.1, U24.1 (1,2EN)
- net A3: now also R17.1, U24.9 (3,4EN)
- net A4: now also R10.1, U25.1 (1,2EN)
- net A5: now also U25.9 (3,4EN)
- net A6: now also U26.1 (1,2EN)
- net A7: now also U26.9 (3,4EN)
- net A8: now also R12.1, U29.1 (1,2EN)
- net A9: now also U29.9 (3,4EN)
- net BUCK_IN: now also U20.7 (V+)
- net BUCK_VOUT: now also U19.4 (AVDD/AVREF), U23.16 (VCC1), U24.16 (VCC1), U25.16 (VCC1), U26.16 (VCC1), U29.16 (VCC1), U30.16 (VCC1)
- net GND: now also R48.2, U19.5 (GND), U20.4 (V-), U23.12 (GND), U23.13 (GND), U23.4 (GND), U23.5 (GND), U24.12 (GND), U24.13 (GND), U24.4 (GND), U24.5 (GND), U25.12 (GND), U25.13 (GND), U25.4 (GND), U25.5 (GND), U26.12 (GND), U26.13 (GND), U26.4 (GND), U26.5 (GND), U29.12 (GND), U29.13 (GND), U29.4 (GND), U29.5 (GND), U30.12 (GND), U30.13 (GND), U30.4 (GND), U30.5 (GND); no longer R10.2, R12.2, R14.2, R16.2, R17.2, R8.2
- net Plate 1.1: now also U23.11 (3Y)
- net Plate 1.2: now also U23.14 (4Y)
- net Plate 10.1: now also U29.3 (1Y)
- net Plate 10.2: now also U29.6 (2Y)
- net Plate 11.1: now also U30.11 (3Y)
- net Plate 11.2: now also U30.14 (4Y)
- net Plate 12.1: now also U30.3 (1Y)
- net Plate 12.2: now also U30.6 (2Y)
- net Plate 2.1: now also U23.3 (1Y)
- net Plate 2.2: now also U23.6 (2Y)
- net Plate 3.1: now also U24.11 (3Y)
- net Plate 3.2: now also U24.14 (4Y)
- net Plate 4.1: now also U24.3 (1Y)
- net Plate 4.2: now also U24.6 (2Y)
- net Plate 5.1: now also U25.11 (3Y)
- net Plate 5.2: now also U25.14 (4Y)
- net Plate 6.1: now also U25.3 (1Y)
- net Plate 6.2: now also U25.6 (2Y)
- net Plate 7.1: now also U26.11 (3Y)
- net Plate 7.2: now also U26.14 (4Y)
- net Plate 8.1: now also U26.3 (1Y)
- net Plate 8.2: now also U26.6 (2Y)
- net Plate 9.1: now also U29.11 (3Y)
- net Plate 9.2: now also U29.14 (4Y)
- net Polarity Enable 1: now also U23.10 (3A), U23.2 (1A), U24.10 (3A), U24.2 (1A), U25.10 (3A), U25.2 (1A), U26.10 (3A), U26.2 (1A), U29.10 (3A), U29.2 (1A), U30.10 (3A), U30.2 (1A)
- net Polarity Enable 2: now also U23.15 (4A), U23.7 (2A), U24.15 (4A), U24.7 (2A), U25.15 (4A), U25.7 (2A), U26.15 (4A), U26.7 (2A), U29.15 (4A), U29.7 (2A), U30.15 (4A), U30.7 (2A)
- net at D10.2 (A): now also R16.2
- net at R19.2: now also D13.2 (A); no longer R17.1
- net at D11.2 (A): now also R17.2
- net at R11.2: now also D5.2 (A); no longer R10.1
- net at R15.2: now also D9.2 (A); no longer R14.1
- net at D4.2 (A): now also R10.2
- net at R18.2: now also D12.2 (A); no longer R16.1
- net at D2.2 (A): now also R8.2
- net at D8.2 (A): now also R14.2
- net at D3.2 (A): now also R9.2
- net MOSI: now reaches U3.11 (MOSI)
- net MOSI: now also U19.3 (DIN)
- net SCK: now reaches U3.13 (SCK)
- net SCK: now also U19.2 (SCLK)
- net SYNC: now reaches U3.26 (A12)
- net SYNC: now also U19.1 (~{SYNC})
- net at R13.2: now also D7.2 (A); no longer R12.1
- net at D6.2 (A): now also R12.2
- new net: R48.1, R49.1, U20.2 (-)
- new net: U19.6 (VOUT), U20.3 (+)
- new net CELL_VOLTAGE: R49.2, U20.6, U23.8 (VCC2), U24.8 (VCC2), U25.8 (VCC2), U26.8 (VCC2), U29.8 (VCC2), U30.8 (VCC2)
- no-connect marks 37 -> 34
Other:
- note added: "Check THT resistor footprint"
- note added: "DAC x Op-Amp"
- note removed: "CAN Bus"
- note removed: "IMPORTANT (README) Some areas need wider traces (marked)"
- note removed: "Op Amps"
- note removed: "TODO: CHECK???"
- moved on the sheet: D1, J1

Commit message: Made Changes but not complete PCB. Gonna reformat
Parts:
- H1, H2, H3, H4: footprint MountingHole:MountingHole_4.3mm_M4_Pad -> MountingHole:MountingHole_2.2mm_M2_DIN965_Pad
- R48, R49: footprint Resistor_THT:R_Bare_Metal_Element_L12.4mm_W4.8mm_P11.40mm -> Resistor_THT:R_Axial_DIN0207_L6.3mm_D2.5mm_P10.16mm_Horizontal
Connections:
- net A0: now also R9.1, U23.9 (3,4EN); no longer R8.1, U23.1 (1,2EN)
- net A1: now also R8.1, U23.1 (1,2EN); no longer R9.1, U23.9 (3,4EN)
- net A2: now also R17.1, U24.9 (3,4EN); no longer R14.1, U24.1 (1,2EN)
- net A3: now also R14.1, U24.1 (1,2EN); no longer R17.1, U24.9 (3,4EN)
- net A4: now also R11.1, U25.9 (3,4EN); no longer R10.1, U25.1 (1,2EN)
- net A5: now also R10.1, U25.1 (1,2EN); no longer R11.1, U25.9 (3,4EN)
- net A6: now also R18.1, U26.9 (3,4EN); no longer R15.1, U26.1 (1,2EN)
- net A7: now also R15.1, U26.1 (1,2EN); no longer R18.1, U26.9 (3,4EN)
- net A8: now also R13.1, U29.9 (3,4EN); no longer R12.1, U29.1 (1,2EN)
- net A9: now also R12.1, U29.1 (1,2EN); no longer R13.1, U29.9 (3,4EN)
- net Plate 11.1: now also U30.6 (2Y); no longer U30.11 (3Y)
- net Plate 11.2: now also U30.3 (1Y); no longer U30.14 (4Y)
- net Plate 12.1: now also U30.14 (4Y); no longer U30.3 (1Y)
- net Plate 12.2: now also U30.11 (3Y); no longer U30.6 (2Y)
- net 3.3v: no longer names the net of U3.3.3V_1 (3.3V), U3.3.3V_2 (3.3V), U3.3.3V_3 (3.3V)
- net RXD: no longer names the net of U3.30 (CRX3)
- net TXD: no longer names the net of U3.31 (CTX3)
- no-connect marks 34 -> 37
Changed lines of the file:
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@@
 	)
 	(no_connect
+		(at 36.83 139.7)
+	)
+	(no_connect
 		(at 36.83 121.92)
 	)
@@
 	)
 	(no_connect
+		(at 77.47 93.98)
+	)
+	(no_connect
 		(at 77.47 104.14)
 	)
@@
 	)
 	(no_connect
+		(at 36.83 142.24)
+	)
+	(no_connect
 		(at 77.47 144.78)
 	)
@@
 		)
 	)
-	(global_label "A1"
+	(global_label "A0"
 		(shape input)
 		(at 153.67 109.22 180)
@@
 		)
 	)
-	(global_label "A0"
+	(global_label "A1"
 		(shape input)
 		(at 135.89 99.06 180)
@@
 		)
 	)
-	(global_label "3.3v"
-		(shape input)
-		(at 77.47 93.98 0)
-		(fields_autoplaced yes)
-		(effects
-			(font
-				(size 1.27 1.27)
-			)
-			(justify left)
-		)
-		(property "Intersheetrefs" "${INTERSHEET_REFS}"
-			(at 84.4466 93.98 0)
-			(effects
-				(font
-					(size 1.27 1.27)
-				)
-				(justify left)
-				(hide yes)
-			)
-		)
-	)
-	(global_label "A7"
+	(global_label "A6"
 		(shape input)
 		(at 285.75 163.83 180)
@@
 	(global_label "Plate 12.1"
 		(shape input)
-		(at 354.33 207.01 0)
+		(at 354.33 219.71 0)
 		(fields_autoplaced yes)
 		(effects
@@
 		)
 		(property "Intersheetrefs" "${INTERSHEET_REFS}"
-			(at 367.4146 207.01 0)
+			(at 367.4146 219.71 0)
 			(effects
 				(font
@@
 		)
 	)
-	(global_label "A3"
+	(global_label "A2"
 		(shape input)
 		(at 285.75 109.22 180)
@@
 		)
 	)
-	(global_label "RXD"
-		(shape input)
-		(at 36.83 139.7 180)
-		(fields_autoplaced yes)
-		(effects
-			(font
-				(size 1.27 1.27)
-			)
-			(justify right)
-		)
-		(property "Intersheetrefs" "${INTERSHEET_REFS}"
-			(at 30.0953 139.7 0)
-			(effects
-				(font
-					(size 1.27 1.27)
-				)
-				(justify right)
-				(hide yes)
-			)
-		)
-	)
 	(global_label "Plate 5.2"
 		(shape input)
@@
 		)
 	)
-	(global_label "A2"
+	(global_label "A3"
 		(shape input)
 		(at 266.7 99.06 180)
@@
 		)
 	)
-	(global_label "A9"
+	(global_label "A8"
 		(shape input)
 		(at 152.4 217.17 180)
@@
 		)
 	)
-	(global_label "A8"
+	(global_label "A9"
 		(shape input)
 		(at 134.62 207.01 180)
@@
 		)
 	)
-	(global_label "A4"
+	(global_label "A5"
 		(shape input)
 		(at 135.89 153.67 180)
@@
 		)
 	)
-	(global_label "A6"
+	(global_label "A7"
 		(shape input)
 		(at 266.7 153.67 180)
@@
 	(global_label "Plate 11.1"
 		(shape input)
-		(at 354.33 217.17 0)
+		(at 354.33 209.55 0)
 		(fields_autoplaced yes)
 		(effects
@@
 		)
 		(property "Intersheetrefs" "${INTERSHEET_REFS}"
-			(at 367.4146 217.17 0)
+			(at 367.4146 209.55 0)
 			(effects
 				(font
@@
 	(global_label "Plate 11.2"
 		(shape input)
-		(at 354.33 219.71 0)
+		(at 354.33 207.01 0)
 		(fields_autoplaced yes)
 		(effects
@@
 		)
 		(property "Intersheetrefs" "${INTERSHEET_REFS}"
-			(at 367.4146 219.71 0)
+			(at 367.4146 207.01 0)
 			(effects
 				(font
@@
 		)
 	)
-	(global_label "A5"
+	(global_label "A4"
 		(shape input)
 		(at 152.4 163.83 180)
@@
 	(global_label "Plate 12.2"
 		(shape input)
-		(at 354.33 209.55 0)
+		(at 354.33 217.17 0)
 		(fields_autoplaced yes)
 		(effects
@@
 		)
 		(property "Intersheetrefs" "${INTERSHEET_REFS}"
-			(at 367.4146 209.55 0)
+			(at 367.4146 217.17 0)
 			(effects
 				(font
@@
 		)
 	)
-	(global_label "TXD"
-		(shape input)
-		(at 36.83 142.24 180)
-		(fields_autoplaced yes)
-		(effects
-			(font
-				(size 1.27 1.27)
-			)
-			(justify right)
-		)
-		(property "Intersheetrefs" "${INTERSHEET_REFS}"
-			(at 30.3977 142.24 0)
-			(effects
-				(font
-					(size 1.27 1.27)
-				)
-				(justify right)
-				(hide yes)
-			)
-		)
-	)
 	(symbol
 		(lib_id "P70-1000045R:P70-1000045R")
@@
 			)
 		)
-		(property "Footprint" "Resistor_THT:R_Bare_Metal_Element_L12.4mm_W4.8mm_P11.40mm"
+		(property "Footprint" "Resistor_THT:R_Axial_DIN0207_L6.3mm_D2.5mm_P10.16mm_Horizontal"
 			(at 46.99 267.97 0)
 			(effects
@@
 			)
 		)
-		(property "Footprint" "MountingHole:MountingHole_4.3mm_M4_Pad"
+		(property "Footprint" "MountingHole:MountingHole_2.2mm_M2_DIN965_Pad"
 			(at 251.46 57.15 0)
 			(effects
@@
 			)
 		)
-		(property "Footprint" "Resistor_THT:R_Bare_Metal_Element_L12.4mm_W4.8mm_P11.40mm"
+		(property "Footprint" "Resistor_THT:R_Axial_DIN0207_L6.3mm_D2.5mm_P10.16mm_Horizontal"
 			(at 54.61 261.62 0)
 			(effects
@@
 			)
 		)
-		(property "Footprint" "MountingHole:MountingHole_4.3mm_M4_Pad"
+		(property "Footprint" "MountingHole:MountingHole_2.2mm_M2_DIN965_Pad"
 			(at 300.99 57.15 0)
 			(effects
@@
 			)
 		)
-		(property "Footprint" "MountingHole:MountingHole_4.3mm_M4_Pad"
+		(property "Footprint" "MountingHole:MountingHole_2.2mm_M2_DIN965_Pad"
 			(at 226.06 57.15 0)
 			(effects
@@
 			)
 		)
-		(property "Footprint" "MountingHole:MountingHole_4.3mm_M4_Pad"
+		(property "Footprint" "MountingHole:MountingHole_2.2mm_M2_DIN965_Pad"
 			(at 275.59 57.15 0)
 			(effects

Commit message: Rerouted PCB layout to actually fit and work. Need to connect Pogo Pins
Parts:
- C8: footprint Capacitor_SMD:C_0201_0603Metric -> Capacitor_SMD:C_0603_1608Metric
Changed lines of the file:
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@@
 			)
 		)
-		(property "Footprint" "Capacitor_SMD:C_0201_0603Metric"
+		(property "Footprint" "Capacitor_SMD:C_0603_1608Metric"
 			(at 354.33 44.45 0)
 			(effects
