File: PCB/FishShocker9000/FishShocker9000.kicad_pcb (KiCad board)
At the start: 2 copper layers, 140 x 285.9 mm, 206 parts, among them J1 Barrel_Jack, J10 P70-1000045R, J100 P70-1000045R, J101 P70-1000045R, J102 P70-1000045R, J103 P70-1000045R, J104 P70-1000045R, J105 P70-1000045R, J106 P70-1000045R, J107 P70-1000045R, J108 P70-1000045R, J109 P70-1000045R, J11 P70-1000045R, J110 P70-1000045R, J111 P70-1000045R, J112 P70-1000045R, J113 P70-1000045R, J114 P70-1000045R, J115 P70-1000045R, J116 P70-1000045R, J117 P70-1000045R, J118 P70-1000045R, J119 P70-1000045R, J12 P70-1000045R, J120 P70-1000045R, J121 P70-1000045R, J122 P70-1000045R, J123 P70-1000045R, J124 P70-1000045R, J125 P70-1000045R, J126 P70-1000045R, J127 P70-1000045R, J128 P70-1000045R, J129 P70-1000045R, J13 P70-1000045R, J130 P70-1000045R, J131 P70-1000045R, J132 P70-1000045R, J133 P70-1000045R, J134 P70-1000045R, J135 P70-1000045R, J136 P70-1000045R, J137 P70-1000045R, J138 P70-1000045R, J139 P70-1000045R, J14 P70-1000045R, J140 P70-1000045R, J141 P70-1000045R, J142 P70-1000045R, J143 P70-1000045R, J144 P70-1000045R, J145 P70-1000045R, J146 Conn_01x03_Pin, J15 P70-1000045R, J16 P70-1000045R, J17 P70-1000045R, J18 P70-1000045R, J19 P70-1000045R, J2 P70-1000045R, J20 P70-1000045R, J21 P70-1000045R, J22 P70-1000045R, J23 P70-1000045R, J24 P70-1000045R, J25 P70-1000045R, J26 P70-1000045R, J27 P70-1000045R, J28 P70-1000045R, J29 P70-1000045R, J3 P70-1000045R, J30 P70-1000045R, J31 P70-1000045R, J32 P70-1000045R, J33 P70-1000045R, J34 P70-1000045R, J35 P70-1000045R, J36 P70-1000045R, J37 P70-1000045R, J38 P70-1000045R, J39 P70-1000045R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

Commit message: Fixed more corruption
Parts:
- J146: footprint Connector_PinHeader_1.00mm:PinHeader_1x03_P1.00mm_Horizontal -> Connector_PinHeader_1.00mm:PinHeader_1x03_P1.00mm_Vertical
- moved J146 0.12 mm to (328.5, 87.0)
Routing:
- net CELL_VOLTAGE: track 129.6 -> 130.7 mm
- net BUCK_IN: track 268.6 -> 269.2 mm

Commit message: Changed pogo pin footprints to connector, fixed routing, removed ferrite bead
Parts:
- removed FB1: 600 @ 600 MHz, Inductor_SMD:L_0805_2012Metric
- J10, J100, J101, J102, J103, J104, J105, J106, J107, J108, J109, J11, J110, J111, J112, J113, J114, J115, J116, J117, J118, J119, J12, J120, J121, J122, J123, J124, J125, J126, J127, J128, J129, J13, J130, J131, J132, J133, J134, J135, J136, J137, J138, J139, J14, J140, J141, J142, J143, J144, J145, J15, J16, J17, J18, J19, J2, J20, J21, J22, J23, J24, J25, J26, J27, J28, J29, J3, J30, J31, J32, J33, J34, J35, J36, J37, J38, J39, J4, J40, J41, J42, J43, J44, J45, J46, J47, J48, J49, J5, J50, J51, J52, J53, J54, J55, J56, J57, J58, J59, J6, J60, J61, J62, J63, J64, J65, J66, J67, J68, J69, J7, J70, J71, J72, J73, J74, J75, J76, J77, J78, J79, J8, J80, J81, J82, J83, J84, J85, J86, J87, J88, J89, J9, J90, J91, J92, J93, J94, J95, J96, J97, J98, J99: footprint Library:HARWIN_P70-1000045R -> Connector_PinHeader_2.54mm:PinHeader_1x01_P2.54mm_Vertical
Connections:
- Q2 pad 3: Net-(Q2-S) -> BUCK_IN
Routing:
- net Net-(Q2-S): track 24.5 -> 0.00 mm
- net Plate 12.1: track 376.2 -> 399.4 mm
- net Plate 8.1: track 351.9 -> 375.0 mm
- net Plate 9.1: track 325.4 -> 347.2 mm
- net Plate 8.2: track 328.6 -> 349.2 mm
- net Plate 9.2: track 280.0 -> 299.6 mm
- net Plate 10.2: track 343.9 -> 363.5 mm
- net Plate 10.1: track 369.8 -> 388.6 mm
- net Plate 12.2: track 351.5 -> 369.4 mm
- net Plate 11.1: track 472.4 -> 490.1 mm
- net Plate 11.2: track 478.4 -> 492.7 mm
- net Plate 1.1: track 161.9 -> 171.4 mm
- net Plate 4.1: track 222.5 -> 218.4 mm
- net Plate 4.2: track 203.5 -> 199.6 mm
- net Plate 2.1: track 167.5 -> 171.3 mm
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